File: hardware/sygeco1.kicad_sch (KiCad schematic)
At the start: 27 parts, among them J1 SSD1306_module, J2 AVR-ISP-6, SW1 SW_Push_DPDT, SW2 SW_Push_DPDT, U1 ATtiny85-20P

Commit message: update symbols + revision
Parts:
- S1: footprint sygeco:SKQUCAA010 -> SKQUCAA010
- U1: footprint sygeco1:dual-dip8-sop8 -> Package_DIP:DIP-8_W7.62mm
Changed lines of the file:
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@@
 	(title_block
 		(title "Sygeco 1")
-		(rev "1.0")
+		(rev "1.2")
 		(company "Sylphide Consulting")
 	)
@@
 			)
 		)
-		(property "Description" ""
+		(property "Description" "Speaker"
 			(at 173.99 83.82 0)
 			(effects
@@
 			)
 		)
-		(property "Description" ""
+		(property "Description" "Single-cell battery"
 			(at 29.21 119.38 0)
 			(effects
@@
 			)
 		)
-		(property "Description" ""
+		(property "Description" "Resistor"
 			(at 157.48 36.83 0)
 			(effects
@@
 			)
 		)
-		(property "Description" ""
+		(property "Description" "Power symbol creates a global label with name \"GND\" , ground"
 			(at 43.18 127 0)
 			(effects
@@
 			)
 		)
-		(property "Description" ""
+		(property "Description" "Power symbol creates a global label with name \"VCC\""
 			(at 52.07 111.76 0)
 			(effects
@@
 			)
 		)
-		(property "Description" ""
+		(property "Description" "Momentary Switch, dual pole double throw"
 			(at 41.91 114.3 0)
 			(effects
@@
 			)
 		)
-		(property "Description" ""
+		(property "Description" "Power symbol creates a global label with name \"GND\" , ground"
 			(at 118.11 93.98 0)
 			(effects
@@
 			)
 		)
-		(property "Description" ""
+		(property "Description" "Momentary Switch, dual pole double throw"
 			(at 156.21 76.2 0)
 			(effects
@@
 			)
 		)
-		(property "Description" ""
+		(property "Description" "Resistor"
 			(at 111.76 39.37 0)
 			(effects
@@
 			)
 		)
-		(property "Description" ""
+		(property "Description" "Resistor"
 			(at 115.57 27.94 0)
 			(effects
@@
 			)
 		)
-		(property "Description" ""
+		(property "Description" "Power symbol creates a global label with name \"VCC\""
 			(at 115.57 24.13 0)
 			(effects
@@
 			)
 		)
-		(property "Datasheet" " ~"
+		(property "Datasheet" "~"
 			(at 33.655 62.23 0)
 			(effects
@@
 			)
 		)
-		(property "Description" ""
+		(property "Description" "Atmel 6-pin ISP connector"
 			(at 66.04 48.26 0)
 			(effects
@@
 			)
 		)
-		(property "Description" ""
+		(property "Description" "Power symbol creates a global label with name \"GND\" , ground"
 			(at 63.5 58.42 0)
 			(effects
@@
 			)
 		)
-		(property "Description" ""
+		(property "Description" "Power symbol creates a global label with name \"VCC\""
 			(at 63.5 35.56 0)
 			(effects
@@
 			)
 		)
-		(property "Description" ""
+		(property "Description" "Resistor"
 			(at 55.88 115.57 0)
 			(effects
@@
 			)
 		)
-		(property "Description" ""
+		(property "Description" "Light emitting diode"
 			(at 55.88 123.19 0)
 			(effects
@@
 			)
 		)
-		(property "Description" ""
+		(property "Description" "Generic connector, single row, 01x04, script generated (kicad-library-utils/schlib/autogen/connector/)"
 			(at 35.56 76.2 0)
 			(effects
@@
 			)
 		)
-		(property "Description" ""
+		(property "Description" "Power symbol creates a global label with name \"GND\" , ground"
 			(at 19.05 81.28 0)
 			(effects
@@
 			)
 		)
-		(property "Description" ""
+		(property "Description" "Power symbol creates a global label with name \"VCC\""
 			(at 19.05 78.74 0)
 			(effects
@@
 			)
 		)
-		(property "Footprint" "sygeco:SKQUCAA010"
+		(property "Footprint" "SKQUCAA010"
 			(at 149.86 38.1 0)
 			(effects
@@
 			)
 		)
-		(property "Description" ""
+		(property "Description" "Unpolarized capacitor"
 			(at 68.58 118.11 0)
 			(effects
@@
 			)
 		)
-		(property "Description" ""
+		(property "Description" "Power symbol creates a global label with name \"GND\" , ground"
 			(at 153.67 45.72 0)
 			(effects
@@
 			)
 		)
-		(property "Description" ""
+		(property "Description" "Power symbol creates a global label with name \"VCC\""
 			(at 157.48 33.02 0)
 			(effects
@@
 			)
 		)
-		(property "Description" ""
+		(property "Description" "Power symbol creates a global label with name \"VCC\""
 			(at 118.11 63.5 0)
 			(effects
@@
 			)
 		)
-		(property "Description" ""
+		(property "Description" "Resistor"
 			(at 119.38 39.37 0)
 			(effects
@@
 			)
 		)
-		(property "Description" ""
+		(property "Description" "Resistor"
 			(at 175.26 27.94 0)
 			(effects
@@
 			)
 		)
-		(property "Description" ""
+		(property "Description" "Power symbol creates a global label with name \"VCC\""
 			(at 175.26 24.13 0)
 			(effects
@@
 			)
 		)
-		(property "Description" ""
+		(property "Description" "Resistor"
 			(at 179.07 39.37 0)
 			(effects
@@
 			)
 		)
-		(property "Description" ""
+		(property "Description" "Resistor"
 			(at 171.45 39.37 0)
 			(effects
@@
 			)
 		)
-		(property "Description" ""
+		(property "Description" "Mounting Hole without connection"
 			(at 20.32 25.4 0)
 			(effects
@@
 			)
 		)
-		(property "Description" ""
+		(property "Description" "Mounting Hole without connection"
 			(at 20.32 30.48 0)
 			(effects
@@
 			)
 		)
-		(property "Description" ""
+		(property "Description" "Light emitting diode"
 			(at 187.96 86.36 0)
 			(effects
@@
 			)
 		)
-		(property "Description" ""
+		(property "Description" "Resistor"
 			(at 187.96 78.74 0)
 			(effects
@@
 			)
 		)
-		(property "Description" ""
+		(property "Description" "Power symbol creates a global label with name \"GND\" , ground"
 			(at 187.96 90.17 0)
 			(effects
@@
 			)
 		)
-		(property "Description" ""
+		(property "Description" "Power symbol creates a global label with name \"VCC\""
 			(at 148.59 63.5 0)
 			(effects
@@
 			)
 		)
-		(property "Description" ""
+		(property "Description" "Power symbol creates a global label with name \"GND\" , ground"
 			(at 168.91 91.44 0)
 			(effects
@@
 			)
 		)
-		(property "Description" ""
+		(property "Description" "Resistor"
 			(at 165.1 83.82 0)
 			(effects
@@
 			)
 		)
-		(property "Footprint" "sygeco1:dual-dip8-sop8"
+		(property "Footprint" "Package_DIP:DIP-8_W7.62mm"
 			(at 118.11 78.74 0)
 			(effects
@@
 			)
 		)
-		(property "Description" ""
+		(property "Description" "20MHz, 8kB Flash, 512B SRAM, 512B EEPROM, debugWIRE, DIP-8"
 			(at 118.11 78.74 0)
 			(effects
@@
 			)
 		)
-		(property "Description" ""
+		(property "Description" "Used to reserve space for rubber pads."
 			(at 30.48 43.18 0)
 			(effects
@@
 			)
 		)
-		(property "Description" ""
+		(property "Description" "Used to reserve space for rubber pads."
 			(at 22.86 50.8 0)
 			(effects
@@
 			)
 		)
-		(property "Description" ""
+		(property "Description" "Used to reserve space for rubber pads."
 			(at 22.86 43.18 0)
 			(effects
@@
 			)
 		)
-		(property "Description" ""
+		(property "Description" "Used to reserve space for rubber pads."
 			(at 30.48 50.8 0)
 			(effects

Commit message: was referencing the old 'sygeco' local symbol library, fixed that to sygeco1
Parts:
- BT1: footprint sygeco:BatteryHolder_China_1x20mm -> sygeco1:BatteryHolder_China_1x20mm
- RP1, RP2, RP3, RP4: footprint sygeco:silicone_rubber_pad -> sygeco1:silicone_rubber_pad
- SW1, SW2: footprint sygeco:DPDT_Switch_with_lock -> sygeco1:DPDT_Switch_with_lock
Changed lines of the file:
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@@
 			)
 		)
-		(property "Footprint" "sygeco:BatteryHolder_China_1x20mm"
+		(property "Footprint" "sygeco1:BatteryHolder_China_1x20mm"
 			(at 29.21 117.856 90)
 			(effects
@@
 			)
 		)
-		(property "Footprint" "sygeco:DPDT_Switch_with_lock"
+		(property "Footprint" "sygeco1:DPDT_Switch_with_lock"
 			(at 41.91 109.22 0)
 			(effects
@@
 			)
 		)
-		(property "Footprint" "sygeco:DPDT_Switch_with_lock"
+		(property "Footprint" "sygeco1:DPDT_Switch_with_lock"
 			(at 156.21 71.12 0)
 			(effects
@@
 			)
 		)
-		(property "Footprint" "sygeco:silicone_rubber_pad"
+		(property "Footprint" "sygeco1:silicone_rubber_pad"
 			(at 30.48 43.18 0)
 			(effects
@@
 			)
 		)
-		(property "Footprint" "sygeco:silicone_rubber_pad"
+		(property "Footprint" "sygeco1:silicone_rubber_pad"
 			(at 22.86 50.8 0)
 			(effects
@@
 			)
 		)
-		(property "Footprint" "sygeco:silicone_rubber_pad"
+		(property "Footprint" "sygeco1:silicone_rubber_pad"
 			(at 22.86 43.18 0)
 			(effects
@@
 			)
 		)
-		(property "Footprint" "sygeco:silicone_rubber_pad"
+		(property "Footprint" "sygeco1:silicone_rubber_pad"
 			(at 30.48 50.8 0)
 			(effects
